File: sb2.brd (EAGLE design)
At the start: 55.5 x 32.4 mm, 31 parts, among them IC1 CP2104, Q1 mmbt2222, Q2 mmbt2222, SW2 KMR2, U1 Si7021-A20, U2 SPX3819, X2 ESP-12

Commit message: update
Parts:
- moved IC1 0.57 mm to (10.4, 8.10)
Routing:
- net GND: track 0.00 -> 199.8 mm, vias 0 -> 5
- net 3.3V: track 0.00 -> 172.4 mm, vias 0 -> 7
- net RESET: track 0.00 -> 88.6 mm, vias 0 -> 3
- net GPIO5/SCL: track 0.00 -> 86.3 mm, vias 0 -> 4
- net GPIO4/SDA: track 0.00 -> 69.9 mm, vias 0 -> 4
- net GPIO12/MISO: track 0.00 -> 62.1 mm, vias 0 -> 3
- net GPIO0: track 0.00 -> 47.5 mm, vias 0 -> 1
- net VBUS: track 0.00 -> 45.2 mm
- net TXD: track 0.00 -> 45.0 mm, vias 0 -> 4
- net GPIO2: track 0.00 -> 44.3 mm
- net CH_PD: track 0.00 -> 42.1 mm
- net GPIO14/SCK: track 0.00 -> 41.8 mm, vias 0 -> 3
- net RXD: track 0.00 -> 28.6 mm, vias 0 -> 3
- net GPIO13/MOSI: track 0.00 -> 28.0 mm, vias 0 -> 2
- net VBAT: track 0.00 -> 26.7 mm
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Other:
- board text removed: "VIN"
