File: sb3.sch (EAGLE design)
At the start: 49 parts, among them IC1 CP2104, Q1 mmbt2222, Q2 mmbt2222, Q3 MMBT2222, Q4 MMBT2222, SW2 KMR2, U1 Si7021-A20, U2 SPX3819, X2 ESP-12, X3 3.5mm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

Commit message: update
Other:
- note added: "ADC"
- note added: "RELAY"
Changed lines of the file:
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@@
 <text x="269.24" y="147.32" size="1.778" layer="94">SET</text>
 <text x="325.12" y="147.32" size="1.778" layer="94">UNSET</text>
+<text x="297.18" y="180.34" size="1.778" layer="94">RELAY</text>
+<text x="302.26" y="60.96" size="1.778" layer="94">ADC</text>
 </plain>
 <instances>
